File: QuadADSR-v1.sch (EAGLE design)
At the start: 73 parts, among them IC1 74AC32D, IC5 MCP6004D, Q1 20MHz, T1 2N3904, T2 2N3904, T3 2N3904, T4 2N3904, U1 ATMEGA328P, U2 DUAL_OPAMP, U3 7805, U4 4051

Commit message: using GMSN! output table
Parts:
- removed CV1, CV2, CV3, CV4: S_JACK, INSTRUO:S_JACK
- removed IC5: MCP6004D, GMSN-R2Project:MCP6004D
- added BUT1, BUT2, BUT3, BUT4: PB6149L-5, INSTRUO:PB6149L-5
- added C18, C20, C22, C3: 560p, rcl:C-USC0805K
- added C19, C21, C23, C6: 47p, rcl:C-USC0805K
- added IC2, IC3: TL074D, linear:TL074D
- added OUTPUT1, OUTPUT2, OUTPUT3, OUTPUT4: S_JACK, INSTRUO:S_JACK
- added R20, R22, R25, R27, R30, R32, R35, R37: 56k, rcl:R-US_R0805
- added R21, R26, R31, R36: 30K, rcl:R-US_R0805
- added R23, R28, R33, R38: 330R, rcl:R-US_R0805
- added R24, R29, R34, R39: 1K, rcl:R-US_R0805
Connections:
- removed net N$13: CV1.TIP, IC5C.-IN, IC5C.OUT
- removed net N$25: CV4.TIP, IC5B.-IN, IC5B.OUT
- removed net N$31: CV3.TIP, IC5A.-IN, IC5A.OUT
- removed net N$36: CV2.TIP, IC5D.-IN, IC5D.OUT
- new net N$16: C3.1, IC2C.+IN, IC2D.+IN, R20.2
- new net N$17: C6.1, IC2C.-IN, R21.1, R22.2
- new net N$23: OUTPUT2.TIP, R21.2, R24.2
- new net N$24: BUT2G$2.A, IC2D.-IN, IC2D.OUT
- new net N$26: BUT2G$2.C, R23.1
- new net N$27: C6.2, IC2C.OUT, R24.1
- new net N$28: C18.1, IC2A.+IN, IC2B.+IN, R25.2
- new net N$29: C19.1, IC2A.-IN, R26.1, R27.2
- new net N$30: OUTPUT1.TIP, R26.2, R29.2
- new net N$32: BUT1G$2.A, IC2B.-IN, IC2B.OUT
- new net N$33: BUT1G$2.C, R28.1
- new net N$34: C19.2, IC2A.OUT, R29.1
- new net N$35: R25.1
- new net N$37: R20.1
- new net N$38: C20.1, IC3A.+IN, IC3B.+IN, R30.2
- new net N$39: C21.1, IC3A.-IN, R31.1, R32.2
- new net N$40: OUTPUT3.TIP, R31.2, R34.2
- new net N$41: BUT3G$2.A, IC3B.-IN, IC3B.OUT
- new net N$42: BUT3G$2.C, R33.1
- new net N$43: C21.2, IC3A.OUT, R34.1
- new net N$44: R30.1
- new net N$45: C22.1, IC3C.+IN, IC3D.+IN, R35.2
- new net N$46: C23.1, IC3C.-IN, R36.1, R37.2
- new net N$47: OUTPUT4.TIP, R36.2, R39.2
- new net N$48: BUT4G$2.A, IC3D.-IN, IC3D.OUT
- new net N$49: BUT4G$2.C, R38.1
- new net N$50: C23.2, IC3C.OUT, R39.1
- new net N$51: R35.1
- net +5V: now also IC2P.V+, IC3P.V+; no longer IC5P.V+
- net GND: now also C18.2, C20.2, C22.2, C3.2, IC2P.V-, IC3P.V-, OUTPUT1.GND, OUTPUT2.GND, OUTPUT3.GND, OUTPUT4.GND, R22.1, R23.2, R27.1, R28.2, R32.1, R33.2, R37.1, R38.2; no longer CV1.GND, CV2.GND, CV3.GND, CV4.GND, IC5P.V-
- net VOUTA: no longer IC5C.+IN
- net VOUTB: no longer IC5D.+IN
- net VOUTC: no longer IC5A.+IN
- net VOUTD: no longer IC5B.+IN

Commit message: removed Switch and checked Schmitt
Parts:
- removed BUT1, BUT2, BUT3, BUT4: PB6149L-5, INSTRUO:PB6149L-5
- removed MODESW: TOGGLE_ON_OFF_ON, INSTRUO:TOGGLE_ON_OFF_ON
- removed R10: 1K, rcl:R-US_R0805
- removed R11, R12: 100K, rcl:R-US_R0805
- removed U2: DUAL_OPAMP, INSTRUO:DUAL_OPAMP
- added C24: 100n, rcl:C-USC0805K
- added C25, C26, C27, C28: 560p, rcl:C-USC0805K
- added IC4: 4093D, 40xx:4093D
- added IC7: 74AC00D, 74xx-eu:74AC00D
- added R40, R42: 10K, rcl:R-US_R0805
- added R41, R43: 1K, rcl:R-US_R0805
- IC1: value 74AC32D -> 4093D; device 74xx-eu:74AC32D -> 40xx:4093D
- R17, R19: value (none) -> 1K; device resistor:R-EU_R0805 -> rcl:R-US_R0805
- R18, R9: value (none) -> 10K; device resistor:R-EU_R0805 -> rcl:R-US_R0805
Connections:
- removed net LED_A: R9.2, U1.PD0(RXD)
- removed net LED_B: R17.2, U1.PD1(TXD)
- removed net LED_C: R18.2, U1.PD3(INT1)
- removed net LED_D: R19.2, U1.PD4(XCK/T0)
- removed net N$12: MODESW.P, R10.1
- removed net N$21: D5.A, R18.1
- removed net N$37: R20.1
- removed net T1: MODESW.S, R11.2, U1.PD6(AIN0)
- removed net T2: MODESW.O, R12.2, U1.PD7(AIN1)
- new net N$31: C26.1, IC1D.O
- new net N$36: IC4A.O, R41.1
- new net N$52: IC1B.O, R43.1
- new net N$54: C28.1, IC4B.O
- new net PULSE1: IC7A.I0, R17.2
- new net PULSE2: IC7A.I1, R19.2
- new net PULSE3: IC7B.I0, R41.2
- new net PULSE4: IC7B.I1, R43.2
- net +12V: now also C15.1, IC2P.V+, IC3P.V+; no longer U2G$3.+12V
- net +5V: now also IC1P.VDD, IC4P.VDD, IC7P.VCC; no longer C15.1, IC1P.VCC, IC2P.V+, IC3P.V+, R10.2
- net -12V: now also C24.2, IC2P.V-, IC3P.V-; no longer U2G$4.-12V
- net GND: now also C24.1, IC1P.VSS, IC4P.VSS, IC7P.GND, R18.1, R40.1, R42.1, R9.1; no longer D3.C, D4.C, D5.C, D6.C, IC1P.GND, IC2P.V-, IC3P.V-, R11.1, R12.1
- net N$11: now also C26.2, IC1C.I0, IC1C.I1, R18.2; no longer IC1A.I1, IC1C.O
- net N$14: now also IC1C.O, R19.1; no longer IC1A.I0, IC1B.O
- net N$19: now also C25.2, IC4C.I0, IC4C.I1, R9.2; no longer D3.A, R9.1
- net N$20: now also IC4C.O; no longer D4.A
- net N$22: now also C25.1, IC4D.O; no longer D6.A, R19.1
- net N$24: now also D4.A; no longer BUT2G$2.A
- net N$26: now also D4.C; no longer BUT2G$2.C
- net N$32: now also D3.A; no longer BUT1G$2.A
- net N$33: now also D3.C; no longer BUT1G$2.C
- net N$35: now also C27.2, IC4A.I0, IC4A.I1, R40.2; no longer R25.1
- net N$41: now also D5.A; no longer BUT3G$2.A
- net N$42: now also D5.C; no longer BUT3G$2.C
- net N$44: now also C27.1, IC1A.O; no longer R30.1
- net N$48: now also D6.A; no longer BUT4G$2.A
- net N$49: now also D6.C; no longer BUT4G$2.C
- net N$51: now also C28.2, IC1B.I0, IC1B.I1, R42.2; no longer R35.1
- net TRIG: now also IC7A.O; no longer IC1A.O
- net TRIG1: now also IC4D.I0, IC4D.I1; no longer IC1C.I1
- net TRIG2: now also IC1D.I0, IC1D.I1, IC7B.O, U1.PD3(INT1); no longer IC1C.I0
- net TRIG3: now also IC1A.I0, IC1A.I1; no longer IC1B.I1
- net TRIG4: now also IC4B.I0, IC4B.I1; no longer IC1B.I0
- net VOUTA: now also R25.1
- net VOUTB: now also R20.1
- net VOUTC: now also R30.1
- net VOUTD: now also R35.1
Other:
- moved on the sheet: IC1P

Commit message: Quad Transistor
Parts:
- removed T1, T2, T3, T4: 2N3904, INSTRUO:TRANSISTOR_MMBT3904
- added U2: MMPQ2222A, Fairchild_By_element14_Batch_1:MMPQ2222A
Connections:
- removed net N$15: R6.1, R7.2, T1.B
- removed net N$3: R2.1, R3.2, T2.B
- removed net N$5: R13.2, R8.1, T3.B
- removed net N$7: R15.1, R16.2, T4.B
- new net B1: R6.1, R7.2, U2.B1
- new net B2: R2.1, R3.2, U2.B2
- new net B3: R13.2, R8.1, U2.B3
- new net B4: R15.1, R16.2, U2.B4
- net GND: now also U2.E1, U2.E2, U2.E3, U2.E4; no longer T1.E, T2.E, T3.E, T4.E
- net TRIG1: now also U2.C1_2; no longer T1.C
- net TRIG2: now also U2.C2_2; no longer T2.C
- net TRIG3: now also U2.C3_2; no longer T3.C
- net TRIG4: now also U2.C4_2; no longer T4.C
